Commit message: JX0: standalone robot description (jx0/description: URDF, MJCF, joint map, meshes) checked against the verified model; 17-joint task with 176 observations for Isaac Lab (Isaac-Velocity-Flat-JX0-Full-v0); policy test suite (speeds, pushes, 60 s endurance, latency), real-time viewer; setup_isaac.bat / train_isaac.bat for the lab PC
Co-Authored-By: Claude Opus 5.5 <noreply@anthropic.com>

File: jx0/description/urdf/jx0.urdf (robot description, URDF)
Before this commit: robot jx0, 21 links, 20 joints
Links:
- link head_link: geometry visual mesh filename=../meshes/JX0_Head.stl scale=0.001 0.001 0.001; visual mesh filename=../meshes/JX0_NeckHub.stl scale=0.001 0.001 0.001
- link left_ankle_pitch_link: geometry visual mesh filename=../meshes/JX0_AnkleBracket_L.stl scale=0.001 0.001 0.001; visual mesh filename=../meshes/JX0_Servo_STS3215.stl scale=0.001 0.001 0.001
- link left_foot_link: geometry collision box size=0.124 0.07 0.002; visual mesh filename=../meshes/JX0_Foot.stl scale=0.001 0.001 0.001
- link left_forearm_link: geometry visual mesh filename=../meshes/JX0_ArmBlade_L.stl scale=0.001 0.001 0.001
- link left_hip_roll_link: geometry visual mesh filename=../meshes/JX0_HipRollBracket_L.stl scale=0.001 0.001 0.001; visual mesh filename=../meshes/JX0_Servo_STS3215.stl scale=0.001 0.001 0.001
- link left_hip_yaw_link: geometry visual mesh filename=../meshes/JX0_HipYawBracket_L.stl scale=0.001 0.001 0.001; visual mesh filename=../meshes/JX0_Servo_STS3215.stl scale=0.001 0.001 0.001
- link left_shin_link: geometry collision mesh filename=../meshes/JX0_Shin_L.stl scale=0.001 0.001 0.001; visual mesh filename=../meshes/JX0_Servo_STS3215.stl scale=0.001 0.001 0.001
- link left_thigh_link: geometry collision mesh filename=../meshes/JX0_Thigh_L.stl scale=0.001 0.001 0.001; visual mesh filename=../meshes/JX0_Servo_STS3215.stl scale=0.001 0.001 0.001
- link left_upper_arm_link: geometry visual mesh filename=../meshes/JX0_Servo_STS3215.stl scale=0.001 0.001 0.001; visual mesh filename=../meshes/JX0_Servo_STS3215.stl scale=0.001 0.001 0.001
- link pelvis: geometry visual mesh filename=../meshes/JX0_Pelvis.stl scale=0.001 0.001 0.001; visual mesh filename=../meshes/JX0_Servo_STS3215.stl scale=0.001 0.001 0.001
- link right_ankle_pitch_link: geometry visual mesh filename=../meshes/JX0_AnkleBracket_R.stl scale=0.001 0.001 0.001; visual mesh filename=../meshes/JX0_Servo_STS3215.stl scale=0.001 0.001 0.001
- link right_foot_link: geometry collision box size=0.124 0.07 0.002; visual mesh filename=../meshes/JX0_Foot.stl scale=0.001 0.001 0.001
- link right_forearm_link: geometry visual mesh filename=../meshes/JX0_ArmBlade_R.stl scale=0.001 0.001 0.001
- link right_hip_roll_link: geometry visual mesh filename=../meshes/JX0_HipRollBracket_R.stl scale=0.001 0.001 0.001; visual mesh filename=../meshes/JX0_Servo_STS3215.stl scale=0.001 0.001 0.001
- link right_hip_yaw_link: geometry visual mesh filename=../meshes/JX0_HipYawBracket_R.stl scale=0.001 0.001 0.001; visual mesh filename=../meshes/JX0_Servo_STS3215.stl scale=0.001 0.001 0.001
- link right_shin_link: geometry collision mesh filename=../meshes/JX0_Shin_R.stl scale=0.001 0.001 0.001; visual mesh filename=../meshes/JX0_Servo_STS3215.stl scale=0.001 0.001 0.001
- link right_thigh_link: geometry collision mesh filename=../meshes/JX0_Thigh_R.stl scale=0.001 0.001 0.001; visual mesh filename=../meshes/JX0_Servo_STS3215.stl scale=0.001 0.001 0.001
- link right_upper_arm_link: geometry visual mesh filename=../meshes/JX0_Servo_STS3215.stl scale=0.001 0.001 0.001; visual mesh filename=../meshes/JX0_Servo_STS3215.stl scale=0.001 0.001 0.001
- link torso_link: geometry visual mesh filename=../meshes/JX0_ChestCap.stl scale=0.001 0.001 0.001; visual mesh filename=../meshes/JX0_Servo_STS3215.stl scale=0.001 0.001 0.001

Commit message: JX0 v0.5: 55 cm with 1.5x longer legs, taller torso, wide visor head (Microban-inspired proportions, own CAD)
- thigh/shin 62/58 -> 93/87 mm, torso +26 mm, arm blades 120 mm; 54.6 cm, 2.99 kg; same 17 STS3215
- head: wide visor head, gloss-black visor (new part JX0_Visor, black PLA) framed by the red neon ring (~188 mm of
  5 x 10 mm strip), ear pods; fixes v0.4's ring channel (the face inside the ring was cut away by build order)
- servo sizing passes (knee 1.26x, hip roll 1.43x); 14/14 gaits; fit, CAD, stops, endurance 12/12, missions 24/24
  (slower bow for the taller body), pushes stay up 100% to 0.72 N s, 83% at 0.96; FEA fatigue SF >= 1.8;
  25/25 software tests (kinematics mass table regenerated); description check pass
- plates re-sliced (blades and black visor on their own plates), verify_plates 0 problems; renders
- the walking policy needs retraining for v0.5 (in progress)

Co-Authored-By: Claude Opus 5.5 <noreply@anthropic.com>

File: jx0/description/urdf/jx0.urdf (robot description, URDF)
Before this commit: robot jx0, 21 links, 20 joints
Links:
- link head_link: geometry visual mesh filename=../meshes/JX0_Head.stl scale=0.001 0.001 0.001; visual mesh filename=../meshes/JX0_NeckHub.stl scale=0.001 0.001 0.001
- link left_shin_link: mass 0.117 -> 0.125
- link left_thigh_link: mass 0.135 -> 0.147
- link right_shin_link: mass 0.117 -> 0.125
- link right_thigh_link: mass 0.135 -> 0.147
- link torso_link: mass 0.663 -> 0.739
Joints:
- joint left_ankle_pitch_joint: origin xyz=0 0 -0.058 rpy=0 0 0 -> xyz=0 0 -0.087 rpy=0 0 0
- joint left_knee_joint: origin xyz=0 0 -0.062 rpy=0 0 0 -> xyz=0 0 -0.093 rpy=0 0 0
- joint left_shoulder_pitch_joint: origin xyz=0.0125 0.063 0.186 rpy=0 0 0 -> xyz=0.0125 0.063 0.212 rpy=0 0 0
- joint neck_yaw_joint: origin xyz=0 0 0.2444 rpy=0 0 0 -> xyz=0 0 0.2704 rpy=0 0 0
- joint right_ankle_pitch_joint: origin xyz=0 0 -0.058 rpy=0 0 0 -> xyz=0 0 -0.087 rpy=0 0 0
- joint right_knee_joint: origin xyz=0 0 -0.062 rpy=0 0 0 -> xyz=0 0 -0.093 rpy=0 0 0
- joint right_shoulder_pitch_joint: origin xyz=0.0125 -0.063 0.186 rpy=0 0 0 -> xyz=0.0125 -0.063 0.212 rpy=0 0 0

Commit message: JX0 head: two WS2812 12-LED ring eyes under clear lenses; all body parts in PETG; walking policy v8
- head 120 mm wide: two 50.8 mm eye pockets for WS2812 12-LED rings (50 mm), a pupil boss that centres each ring,
  a wire slot behind each ring so the wiring runs inside the head and down the neck hub (nothing in front), mic holes
  between the eyes; new part JX0_EyeLens x2 (1.2 mm clear PETG); the neon channel and visor are gone; 157 g
- jx0bot/eyes.py: the rings on SPI GPIO 10 (I2S has 18-21), brightness cap 0.3 (~0.5 A), states idle / listening /
  thinking / speaking with blinks, moods via a new Claude tool "eyes"; main.py drives them; tests 26/26
- print: body plates in PETG (white, 3 walls 25 %: new PETG-body profile), lenses in clear PETG; verify_plates 0
  problems: 707 g grey + 585 g white
- run_all passes (knee 1.20x, hip roll 1.39x; 14/14 gaits; fit; CAD; stops; missions 24/24; endurance 12/12; FEA
  fatigue SF >= 1.5 at the yaw keeper (was 2.0); description); jx0_walk17_v8 passes the suite (11/11, 96/96,
  endurance, latency) and the clearance check (1700 poses, 0 contacts)
- docs: build guide (eyes assembly), wiring (GPIO 10, power), print README, renders

Co-Authored-By: Claude Opus 5.5 <noreply@anthropic.com>

File: jx0/description/urdf/jx0.urdf (robot description, URDF)
Before this commit: robot jx0, 21 links, 20 joints
Links:
- link head_link: geometry visual mesh filename=../meshes/JX0_EyeLens.stl scale=0.001 0.001 0.001; visual mesh filename=../meshes/JX0_EyeLens.stl scale=0.001 0.001 0.001
- link torso_link: mass 0.739 -> 0.796

Commit message: JX0: stronger hip-yaw keeper and bracket; chest webcam mount and recorder
- yaw keeper: arc to 125 deg (the swinging longer leg tilted the disc past 104 deg, loading the lip to the 100 N cap in
  normal walking), 5 M2 x 10 screws, outer wall to r 26, lip corners relieved where the thigh / hip-roll bracket pass;
  fatigue SF 1.5 -> 1.9, pelvis 1.9 -> 3.0; hip-yaw bracket: fillets in its two inside corners, 1.6 -> 1.7
- chest camera: 20 mm window in the torso front under the lettering, two shelves inside for a USB webcam head
  (Lapcare Lapcam ~85 x 35 x 25 mm), JX0_CamClamp plate with 4 M2 x 10 CSK; webcam keep-out in the fit/CAD checks;
  assembly step; jx0bot/camera.py records 5-minute MP4 segments while the program runs (OpenCV), test
- run_all passes (knee 1.18x, hip roll 1.38x; 14/14 gaits; fit 188 screws reachable; CAD; stops 0 problems;
  missions 24/24; endurance 12/12; FEA fatigue SF >= 1.7; 27/27 tests; description); jx0_walk17_v8 passes the suite
  and the clearance check on the 3.10 kg robot; plates 0 problems

Co-Authored-By: Claude Opus 5.5 <noreply@anthropic.com>

File: jx0/description/urdf/jx0.urdf (robot description, URDF)
Before this commit: robot jx0, 21 links, 20 joints
Links:
- link torso_link: mass 0.796 -> 0.846; geometry visual mesh filename=../meshes/JX0_CamClamp.stl scale=0.001 0.001 0.001; visual mesh filename=../meshes/JX0_ChestCap.stl scale=0.001 0.001 0.001

Commit message: JX0 battery: 3S 2200 stands in a floor pocket in the middle of the torso, leads out a 9 mm hole in the back wall
Battery placement study (servo sizing + walking sim + voxel FEA of the yaw keeper and hip-yaw bracket):
the 306 g 4400 mAh pack drops the yaw keeper's fatigue SF from 1.9 to 1.2 wherever it goes, and hung on the back
it takes the knee under its continuous rating (0.96x). The 2200 standing in the middle keeps the committed margins:
knee 1.18x / 1.11x continuous, keeper 1.9, hip-yaw bracket 1.7. Fit 186 screws OK, CAD 0 clashes (1373 poses),
plates 0 problems, policy v8 passes sim2sim, description check passes.

Co-Authored-By: Claude Opus 5.5 <noreply@anthropic.com>

File: jx0/description/urdf/jx0.urdf (robot description, URDF)
Before this commit: robot jx0, 21 links, 20 joints
Links:
- link torso_link: mass 0.846 -> 0.852
